File: hardware/FT02_PowerBoard_V1/08_3V3_BUCKBOOST.kicad_sch (KiCad schematic)
At the start: 7 parts, among them U801 TPS63802DLAR

Commit message: Wire FT02 Phase 1 power stages and verify partial shunt boundary
Connections:
- net SYS_RAW: no longer U801.1 (EN)
- new net RAIL_PERMIT: U801.1 (EN)
Other:
- note added: "EN=RAIL_PERMIT from U702: automatic system UVLO, nominal3.30V. Battery cutoff and rebound NOT qualified."
- note removed: "EN tied to SYS_RAW: default-on reference only. Rail-disable and system UVLO not yet implemented."
